File: tardigrade_uart_bridge/mcu.kicad_sch (KiCad schematic)
At the start: 1 part, among them U1 ATmega328P-A

Commit message: overview
Changed lines of the file:
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@@
+		)
+	)
+	(hierarchical_label "CONTROL_5V"
+		(shape input)
+		(at 130.81 115.57 0)
+		(effects
+			(font
+				(size 1.27 1.27)
+			)
+			(justify left)
 		)
 	)
@@
 		)
 	)
+	(hierarchical_label "CONTROL_KILL"
+		(shape input)
+		(at 130.81 123.19 0)
+		(effects
+			(font
+				(size 1.27 1.27)
+			)
+			(justify left)
+		)
+	)
 	(hierarchical_label "ICSP_MOSI"
 		(shape input)
@@
 		)
 	)
+	(hierarchical_label "PROBE_KILL"
+		(shape input)
+		(at 132.08 128.27 0)
+		(effects
+			(font
+				(size 1.27 1.27)
+			)
+			(justify left)
+		)
+	)
 	(hierarchical_label "UART_RX"
 		(shape input)
-		(at 132.08 104.14 0)
+		(at 130.81 109.22 0)
 		(effects
 			(font
@@
 		)
 	)
+	(hierarchical_label "CONTROL_3.3V"
+		(shape input)
+		(at 130.81 119.38 0)
+		(effects
+			(font
+				(size 1.27 1.27)
+			)
+			(justify left)
+		)
+	)
 	(hierarchical_label "UART_TX"
 		(shape input)
-		(at 132.08 100.33 0)
+		(at 130.81 105.41 0)
 		(effects
 			(font

Commit message: added basic passives for mcu
Parts:
- added C1, C2: 100nF, symbol Device:C
- added C3, C4: C, symbol Device:C
- added R1: 1M, symbol Device:R_US
- added Y1: Crystal, symbol Device:Crystal
Connections:
- net GND: now also C1.1, C2.2, C3.2, C4.2
- net 3.3V: now reaches U1.18 (AVCC)
- net 3.3V: now also U1.4 (VCC), U1.6 (VCC), C1.2, C2.1
- net MCU_RESET: now reaches U1.29 (~{RESET}/PC6)
- net XTAL1: now reaches U1.7 (XTAL1/PB6)
- net XTAL1: now also C4.1, R1.1, Y1.1
- net XTAL2: now reaches U1.8 (XTAL2/PB7)
- net XTAL2: now also C3.1, R1.2, Y1.2
Other:
- moved on the sheet: U1
