File: tardigrade_uart_bridge/tardigrade_uart_bridge.kicad_sch (KiCad schematic)
At the start: 0 parts

Commit message: overview
Parts:
- added J1: Conn_01x08_Socket, symbol Connector:Conn_01x08_Socket
- added J2: Conn_01x03_Socket, symbol Connector:Conn_01x03_Socket
- added J3, J4: Conn_01x02_Socket, symbol Connector:Conn_01x02_Socket
Connections:
- new net GND: J1.1 (Pin_1), J2.1 (Pin_1), J3.1 (Pin_1), J4.1 (Pin_1)
Other:
- sheet mcu ports: added CONTROL_3.3V, CONTROL_5V, CONTROL_KILL, I2C_SCL, I2C_SDA, ICSP_CS, ICSP_MISO, ICSP_MOSI, ICSP_SCK, PROBE_KILL, PWM_0, PWM_1, PWM_2, PWM_3, PWM_4, PWM_5, UART_RX, UART_TX; removed none
- note added: "Power In"
- note added: "Power Out"
- note added: "TO ESC Stack"
- note added: "To Host"

Commit message: added basic passives for mcu
Parts:
- added J5: Conn_01x05_Socket, symbol Connector:Conn_01x05_Socket
Connections:
- net GND: now also J5.1 (Pin_1)
Other:
- sheet mcu ports: added MCU_RESET; removed none
- note added: "Program"
Changed lines of the file:
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@@
+		)
+	)
+	(rectangle
+		(start 140.97 140.97)
+		(end 180.34 158.75)
+		(stroke
+			(width 0)
+			(type default)
+		)
+		(fill
+			(type none)
 		)
 	)
@@
 		(exclude_from_sim no)
 		(at 214.122 80.518 0)
+		(effects
+			(font
+				(size 1.27 1.27)
+			)
+		)
+	)
+	(text "Program"
+		(exclude_from_sim no)
+		(at 145.288 143.256 0)
 		(effects
 			(font
@@
 		)
 	)
+	(symbol
+		(lib_id "power:GND")
+		(at 166.37 144.78 270)
+		(unit 1)
+		(exclude_from_sim no)
+		(in_bom yes)
+		(on_board yes)
+		(dnp no)
+		(fields_autoplaced yes)
+		(property "Reference" "#PWR010"
+			(at 160.02 144.78 0)
+			(effects
+				(font
+					(size 1.27 1.27)
+				)
+				(hide yes)
+			)
+		)
+		(property "Value" "GND"
+			(at 162.56 144.7799 90)
+			(effects
+				(font
+					(size 1.27 1.27)
+				)
+				(justify right)
+			)
+		)
+		(property "Footprint" ""
+			(at 166.37 144.78 0)
+			(effects
+				(font
+					(size 1.27 1.27)
+				)
+				(hide yes)
+			)
+		)
+		(property "Datasheet" ""
+			(at 166.37 144.78 0)
+			(effects
+				(font
+					(size 1.27 1.27)
+				)
+				(hide yes)
+			)
+		)
+		(property "Description" "Power symbol creates a global label with name \"GND\" , ground"
+			(at 166.37 144.78 0)
+			(effects
+				(font
+					(size 1.27 1.27)
+				)
+				(hide yes)
+			)
+		)
+		(pin "1"
+		)
+		(instances
+			(project "tardigrade_uart_bridge"
+				(path "/57ceeace-a0a4-4368-ac37-c710a76ecbf9"
+					(reference "#PWR010")
+					(unit 1)
+				)
+			)
+		)
+	)
+	(symbol
+		(lib_id "Connector:Conn_01x05_Socket")
+		(at 171.45 149.86 0)
+		(unit 1)
+		(exclude_from_sim no)
+		(in_bom yes)
+		(on_board yes)
+		(dnp no)
+		(fields_autoplaced yes)
+		(property "Reference" "J5"
+			(at 172.72 148.5899 0)
+			(effects
+				(font
+					(size 1.27 1.27)
+				)
+				(justify left)
+			)
+		)
+		(property "Value" "Conn_01x05_Socket"
+			(at 172.72 151.1299 0)
+			(effects
+				(font
+					(size 1.27 1.27)
+				)
+				(justify left)
+			)
+		)
+		(property "Footprint" ""
+			(at 171.45 149.86 0)
+			(effects
+				(font
+					(size 1.27 1.27)
+				)
+				(hide yes)
+			)
+		)
+		(property "Datasheet" "~"
+			(at 171.45 149.86 0)
+			(effects
+				(font
+					(size 1.27 1.27)
+				)
+				(hide yes)
+			)
+		)
+		(property "Description" "Generic connector, single row, 01x05, script generated"
+			(at 171.45 149.86 0)
+			(effects
+				(font
+					(size 1.27 1.27)
+				)
+				(hide yes)
+			)
+		)
+		(pin "5"
+		)
+		(pin "4"
+		)
+		(pin "3"
+		)
+		(pin "2"
+		)
+		(pin "1"
+		)
+		(instances
+			(project ""
+				(path "/57ceeace-a0a4-4368-ac37-c710a76ecbf9"
+					(reference "J5")
+					(unit 1)
+				)
+			)
+		)
+	)
 	(sheet
 		(at 33.02 30.48)
@@
 			)
 		)
+		(pin "MCU_RESET" input
+			(at 33.02 91.44 180)
+			(effects
+				(font
+					(size 1.27 1.27)
+				)
+				(justify left)
+			)
+		)
