File: mcu.kicad_sch (KiCad schematic)
At the start: 7 parts, among them U1 ATmega328P-A, Y1 Crystal

Commit message: added peripheral connectors, started PCB
Parts:
- C1, C2, R1: footprint (none) -> Capacitor_SMD:C_0805_2012Metric_Pad1.18x1.45mm_HandSolder
- C3, C4: value C -> 22pF; footprint (none) -> Capacitor_SMD:C_0805_2012Metric_Pad1.18x1.45mm_HandSolder
- Y1: footprint (none) -> Crystal:Crystal_HC49-U_Vertical
Changed lines of the file:
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@@
 			)
 		)
-		(property "Footprint" ""
+		(property "Footprint" "Capacitor_SMD:C_0805_2012Metric_Pad1.18x1.45mm_HandSolder"
 			(at 30.734 84.074 90)
 			(effects
@@
 			)
 		)
-		(property "Footprint" ""
+		(property "Footprint" "Capacitor_SMD:C_0805_2012Metric_Pad1.18x1.45mm_HandSolder"
 			(at 85.09 43.4848 0)
 			(effects
@@
 		(on_board yes)
 		(dnp no)
-		(fields_autoplaced yes)
 		(property "Reference" "Y1"
-			(at 31.7501 97.79 90)
-			(effects
-				(font
-					(size 1.27 1.27)
-				)
-				(justify right)
+			(at 35.052 92.456 0)
+			(effects
+				(font
+					(size 1.27 1.27)
+				)
+				(justify left)
 			)
 		)
 		(property "Value" "Crystal"
-			(at 29.2101 97.79 90)
-			(effects
-				(font
-					(size 1.27 1.27)
-				)
-				(justify right)
-			)
-		)
-		(property "Footprint" ""
+			(at 35.052 94.996 0)
+			(effects
+				(font
+					(size 1.27 1.27)
+				)
+				(justify left)
+			)
+		)
+		(property "Footprint" "Crystal:Crystal_HC49-U_Vertical"
 			(at 30.48 93.98 0)
 			(effects
@@
 			)
 		)
-		(property "Footprint" ""
+		(property "Footprint" "Capacitor_SMD:C_0805_2012Metric_Pad1.18x1.45mm_HandSolder"
 			(at 67.0052 44.45 0)
 			(effects
@@
 			)
 		)
-		(property "Value" "C"
+		(property "Value" "22pF"
 			(at 19.812 100.584 90)
 			(effects
@@
 			)
 		)
-		(property "Footprint" ""
+		(property "Footprint" "Capacitor_SMD:C_0805_2012Metric_Pad1.18x1.45mm_HandSolder"
 			(at 27.6352 104.14 0)
 			(effects
@@
 			)
 		)
-		(property "Value" "C"
+		(property "Value" "22pF"
 			(at 39.37 100.33 90)
 			(effects
@@
 			)
 		)
-		(property "Footprint" ""
+		(property "Footprint" "Capacitor_SMD:C_0805_2012Metric_Pad1.18x1.45mm_HandSolder"
 			(at 35.2552 104.14 0)
 			(effects

Commit message: added pwm outputs, power connectors, etc.
Connections:
- net I2C_SCL: now also U1.28 (PC5)
- net I2C_SDA: now also U1.27 (PC4)
- net ICSP_MISO: now also U1.16 (PB4)
- net ICSP_MOSI: now also U1.15 (PB3)
- net ICSP_SCK: now also U1.17 (PB5)
- net PWM_0: now also U1.10 (PD6)
- net PWM_1: now also U1.9 (PD5)
- net PWM_2: now also U1.13 (PB1)
- net PWM_3: now also U1.14 (PB2)
- net PWM_5: now also U1.1 (PD3)
- net UART_RX: now also U1.31 (PD1)
- net UART_TX: now also U1.30 (PD0)
